Commit message: mapping setting

File: src/kora_k3/urdf/k3.xacro (robot description, xacro)
@@ -143,8 +143,8 @@
     <joint name = "laser_joint" type = "fixed">
         <parent link = "base_link"/>
-        <child link = "laser_frame"/>
+        <child link = "laser"/>
         <origin xyz = "0 0 0.075" rpy="0 0 0"/>
     </joint>
-    <link name="laser_frame">
+    <link name="laser">
         <visual>
             <geometry>
@@ -186,5 +186,5 @@
     </link>
     <!-- IMU -->
-    <joint name = "imu_link" type = "fixed">
+    <joint name = "imu_joint" type = "fixed">
         <parent link = "body"/>
         <child link = "imu_link"/>

Commit message: k3 urdf revision and IMU filtering

File: src/kora_k3/urdf/k3.xacro (robot description, xacro)
@@ -23,5 +23,5 @@
         <parent link = "base_link"/>
         <child link = "body" />
-        <origin xyz = "-0.12 0 0"/>
+        <origin xyz = "-0.1514 0 -0.05"/>
     </joint>
     <link name = "body">
@@ -29,5 +29,5 @@
             <origin xyz = "0.1 0 0.03"/>
             <geometry>
-                <box size = "0.2 0.1 0.06"/>
+                <box size = "0.425 0.23 0.15"/>
             </geometry>
             <material name = "white"/>
@@ -36,8 +36,8 @@
             <origin xyz = "0.1 0 0.03"/>
             <geometry>
-                <box size = "0.2 0.1 0.06"/>
-            </geometry>
-        </collision>
-        <xacro:inertial_box mass="0.5" x="0.2" y="0.1" z="0.06">
+                <box size = "0.425 0.23 0.15"/>
+            </geometry>
+        </collision>
+        <xacro:inertial_box mass="3.5" x="0.425" y="0.23" z="0.15">
             <origin xyz="0.1 0 0.03" rpy="0 0 0"/>
         </xacro:inertial_box>
@@ -78,5 +78,5 @@
         <parent link="base_link"/>
         <child  link="front_left_steer_link"/>
-        <origin xyz="0.055 0.065 0" rpy="0 0 0"/>   <!-- 원래 앞바퀴 위치와 같게 -->
+        <origin xyz="0.1736 0.115 -0.05" rpy="0 0 0"/>   <!-- 원래 앞바퀴 위치와 같게 -->
         <axis xyz="0 0 1"/>
         <limit lower="-0.349066" upper="0.349066" effort="30" velocity="2.0"/>
@@ -85,5 +85,5 @@
         <parent link="base_link"/>
         <child  link="front_right_steer_link"/>
-        <origin xyz="0.055 -0.065 0" rpy="0 0 0"/>
+        <origin xyz="0.1736 -0.115 -0.05" rpy="0 0 0"/>
         <axis xyz="0 0 1"/>
         <limit lower="-0.349066" upper="0.349066" effort="30" velocity="2.0"/>
@@ -103,5 +103,5 @@
     <!-- REAR LEFT WHEEL -->
     <xacro:wheel_link name="rear_left_wheel" parent_link="base_link"
-                  xyz="-0.1 0.065 0" rpy="-${pi/2} 0 0" direction="1"/>
+                  xyz="-0.1514 0.115 -0.05" rpy="-${pi/2} 0 0" direction="1"/>
     <gazebo reference = "rear_left_wheel">
         <material>Gazebo/Black</material>
@@ -109,5 +109,5 @@
     <!-- REAR RIGHT WHEEL -->
     <xacro:wheel_link name="rear_right_wheel" parent_link="base_link"
-                  xyz="-0.1 -0.065 0" rpy="${pi/2} 0 0" direction="-1"/>
+                  xyz="-0.1514 -0.115 -0.05" rpy="${pi/2} 0 0" direction="-1"/>
     <gazebo reference = "rear_right_wheel">
         <material>Gazebo/Black</material>
@@ -144,10 +144,10 @@
         <parent link = "base_link"/>
         <child link = "laser"/>
-        <origin xyz = "0 0 0.075" rpy="0 0 0"/>
+        <origin xyz = "0.0836 0 0.11" rpy="0 0 0"/>
     </joint>
     <link name="laser">
         <visual>
             <geometry>
-                <cylinder radius="0.03" length="0.03"/>
+                <cylinder radius="0.02" length="0.04"/>
             </geometry>
             <material name = "red"/>
@@ -155,5 +155,5 @@
         <collision>
             <geometry>
-                <cylinder radius="0.03" length="0.03"/>
+                <cylinder radius="0.02" length="0.04"/>
             </geometry>
         </collision>
@@ -161,12 +161,12 @@
     <!-- CAMERA -->
     <joint name = "camera_joint" type = "fixed">
-        <parent link = "body"/>
+        <parent link = "base_link"/>
         <child link = "camera_link"/>
-        <origin xyz = "0.20 0 0.03" rpy="0 0 0"/>
+        <origin xyz = "0.1286 0 0.06" rpy="0 0 0"/>
     </joint>
     <link name = "camera_link">
         <visual>
             <geometry>
-                <box size = "0.01 0.03 0.03"/>
+                <box size = "0.025 0.12 0.03"/>
             </geometry>
             <material name = "red"/>
@@ -174,9 +174,9 @@
         <collision>
             <geometry>
-                <box size = "0.01 0.03 0.03"/>
-            </geometry>
-        </collision>
-    </link>
-    <joint name = "camera_optical_joint" type = "fixed">
+                <box size = "0.025 0.12 0.03"/>
+            </geometry>
+        </collision>
+    </link>
+    <!-- <joint name = "camera_optical_joint" type = "fixed">
         <parent link = "camera_link"/>
         <child link = "camera_link_optical"/>
@@ -184,10 +184,10 @@
     </joint>
     <link name = "camera_link_optical">
-    </link>
+    </link> -->
     <!-- IMU -->
     <joint name = "imu_joint" type = "fixed">
-        <parent link = "body"/>
+        <parent link = "base_link"/>
         <child link = "imu_link"/>
-        <origin xyz = "0.03 0 0.065" rpy = "0 0 0"/>
+        <origin xyz = "-0.1014 0 0.02" rpy = "0 0 0"/>
     </joint>
     <link name = "imu_link">
@@ -200,5 +200,5 @@
         <collision>
             <geometry>
-                <box size = "0.03 0.01 0.03"/>
+                <box size = "0.03 0.03 0.01"/>
             </geometry>
         </collision>

File: src/kora_k3/urdf/macros.xacro (robot description, xacro)
@@ -40,5 +40,5 @@
                 <origin xyz="0 0 0" rpy="${rpy}"/>
                 <geometry>
-                    <cylinder radius="0.03" length="0.03"/>
+                    <cylinder radius="0.05" length="0.04"/>
                 </geometry>
                 <material name="black"/>
@@ -47,8 +47,8 @@
                 <origin xyz="0 0 0" rpy="${rpy}"/>
                 <geometry>
-                    <cylinder radius="0.03" length="0.03"/>
+                    <cylinder radius="0.05" length="0.04"/>
                 </geometry>
             </collision>
-            <xacro:inertial_cylinder mass="0.1" length="0.03" radius="0.03">
+            <xacro:inertial_cylinder mass="0.1" length="0.04" radius="0.05">
                 <origin xyz="0 0 0" rpy="0 0 0"/>
             </xacro:inertial_cylinder>
